File: pcb/draft.kicad_pcb (KiCad board)
At the start: 2 copper layers, 109 x 54 mm, 60 parts, among them J1 MALE, J10 TC2030_NL, J101 MALE, J102 FEMALE, J103 MALE, J104 FEMALE, J105 MALE, J106 FEMALE, J107 MALE, J108 FEMALE, J11 STANDOFF, J111 STANDOFF, J112 STANDOFF, J113 STANDOFF, J114 STANDOFF, J12 STANDOFF, J13 STANDOFF, J14 STANDOFF, J2 FEMALE, J3 MALE, J4 FEMALE, J5 MALE, J6 FEMALE, J7 MALE, J8 FEMALE, J9 DTR, Q1 2N3904, SW1 ACTION, SW2 ACTION, SW3 ACTION, SW4 ACTION, U3 ATmega328P-MU, Y1 YSX321SL

Commit message: Add footprint for diode
Parts:
- moved C1 30.0 mm to (118.4, 108.7)
- moved Y1 27.2 mm to (115.7, 109.6)
- moved C2 25.6 mm to (116.9, 107.2)
- moved R7 3.26 mm to (112.0, 114.6)
- moved R8 1.23 mm to (115.3, 113.8)
Changed lines of the file:
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@@
   )
   (module Resistor_SMD:R_0402_1005Metric (layer F.Cu)
-    (at 112.35 111.312)
+    (at 112.037 114.554)
     (descr "Resistor SMD 0402 (1005 Metric), square (rectangular) end terminal, IPC_7351 nominal, (Body size source: http://www.tortai-tech.com/upload/download/2011102023233369053.pdf), generated with kicad-footprint-generator")
     (tags resistor)
@@
   )
   (module Resistor_SMD:R_0402_1005Metric (layer F.Cu)
-    (at 115.144 112.582)
+    (at 115.339 113.792)
     (descr "Resistor SMD 0402 (1005 Metric), square (rectangular) end terminal, IPC_7351 nominal, (Body size source: http://www.tortai-tech.com/upload/download/2011102023233369053.pdf), generated with kicad-footprint-generator")
     (tags resistor)
@@
   )
   (module Capacitor_SMD:C_0402_1005Metric (layer F.Cu)
-    (at 88.441001 106.299001)
+    (at 118.392 108.712)
     (descr "Capacitor SMD 0402 (1005 Metric), square (rectangular) end terminal, IPC_7351 nominal, (Body size source: IPC-SM-782 page 76, https://www.pcb-3d.com/wordpress/wp-content/uploads/ipc-sm-782a_amendment_1_and_2.pdf), generated with kicad-footprint-generator")
     (tags capacitor)
@@
   )
   (module Capacitor_SMD:C_0402_1005Metric (layer F.Cu)
-    (at 91.311001 106.449001)
+    (at 116.868 107.188)
     (descr "Capacitor SMD 0402 (1005 Metric), square (rectangular) end terminal, IPC_7351 nominal, (Body size source: IPC-SM-782 page 76, https://www.pcb-3d.com/wordpress/wp-content/uploads/ipc-sm-782a_amendment_1_and_2.pdf), generated with kicad-footprint-generator")
     (tags capacitor)
@@
   )
   (module node:YSX321SL (layer F.Cu)
-    (at 89.306 103.364)
+    (at 115.74 109.64)
     (fp_text reference Y1 (at 0 -2.286) (layer F.SilkS)
       (effects (font (size 1 1) (thickness 0.15)))

Commit message: Place footprints
Parts:
- added BZ1: Buzzer, node:MLT-5020, F.Cu at (143.2, 59.3)
- added D5: 1N4148, Diode_SMD:D_SOD-323, F.Cu at (149.3, 57.6)
Changed lines of the file:
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@@
     (tracks 29)
     (zones 0)
-    (modules 60)
+    (modules 62)
     (nets 73)
   )
@@
       (at (xyz 0 0 0))
       (scale (xyz 1 1 1))
+      (rotate (xyz 0 0 0))
+    )
+  )
+  (module node:MLT-5020 (layer F.Cu)
+    (at 143.2 59.302001)
+    (fp_text reference BZ1 (at 0 -3.4) (layer F.SilkS)
+      (effects (font (size 1 1) (thickness 0.15)))
+    )
+    (fp_text value Buzzer (at 0 3.6) (layer F.Fab)
+      (effects (font (size 1 1) (thickness 0.15)))
+    )
+    (fp_line (start -2.6 -2.6) (end -2.6 2.6) (layer F.Fab) (width 0.12))
+    (fp_line (start 2.6 -2.6) (end 2.6 2.6) (layer F.Fab) (width 0.12))
+    (fp_line (start -2.6 -2.6) (end 2.6 -2.6) (layer F.Fab) (width 0.12))
+    (fp_line (start 2.6 2.6) (end -2.6 2.6) (layer F.Fab) (width 0.12))
+    (pad 3 smd rect (at -2.5 -1.7 90) (size 1 2) (layers F.Cu F.Paste F.Mask))
+    (pad 2 smd rect (at -2.5 1.7 90) (size 1 2) (layers F.Cu F.Paste F.Mask)
+      (net 70 "Net-(BZ1-Pad2)"))
+    (pad 1 smd rect (at 2.5 1.7 90) (size 1 2) (layers F.Cu F.Paste F.Mask)
+      (net 72 "Net-(BZ1-Pad1)"))
+  )
+  (module Diode_SMD:D_SOD-323 (layer F.Cu)
+    (at 149.325001 57.617001)
+    (descr SOD-323)
+    (tags SOD-323)
+    (attr smd)
+    (fp_text reference D5 (at 0 -1.85) (layer F.SilkS)
+      (effects (font (size 1 1) (thickness 0.15)))
+    )
+    (fp_text value 1N4148 (at 0.1 1.9) (layer F.Fab)
+      (effects (font (size 1 1) (thickness 0.15)))
+    )
+    (fp_line (start -1.5 -0.85) (end 1.05 -0.85) (layer F.SilkS) (width 0.12))
+    (fp_line (start -1.5 0.85) (end 1.05 0.85) (layer F.SilkS) (width 0.12))
+    (fp_line (start -1.6 -0.95) (end -1.6 0.95) (layer F.CrtYd) (width 0.05))
+    (fp_line (start -1.6 0.95) (end 1.6 0.95) (layer F.CrtYd) (width 0.05))
+    (fp_line (start 1.6 -0.95) (end 1.6 0.95) (layer F.CrtYd) (width 0.05))
+    (fp_line (start -1.6 -0.95) (end 1.6 -0.95) (layer F.CrtYd) (width 0.05))
+    (fp_line (start -0.9 -0.7) (end 0.9 -0.7) (layer F.Fab) (width 0.1))
+    (fp_line (start 0.9 -0.7) (end 0.9 0.7) (layer F.Fab) (width 0.1))
+    (fp_line (start 0.9 0.7) (end -0.9 0.7) (layer F.Fab) (width 0.1))
+    (fp_line (start -0.9 0.7) (end -0.9 -0.7) (layer F.Fab) (width 0.1))
+    (fp_line (start -0.3 -0.35) (end -0.3 0.35) (layer F.Fab) (width 0.1))
+    (fp_line (start -0.3 0) (end -0.5 0) (layer F.Fab) (width 0.1))
+    (fp_line (start -0.3 0) (end 0.2 -0.35) (layer F.Fab) (width 0.1))
+    (fp_line (start 0.2 -0.35) (end 0.2 0.35) (layer F.Fab) (width 0.1))
+    (fp_line (start 0.2 0.35) (end -0.3 0) (layer F.Fab) (width 0.1))
+    (fp_line (start 0.2 0) (end 0.45 0) (layer F.Fab) (width 0.1))
+    (fp_line (start -1.5 -0.85) (end -1.5 0.85) (layer F.SilkS) (width 0.12))
+    (fp_text user %R (at 0 -1.85) (layer F.Fab)
+      (effects (font (size 1 1) (thickness 0.15)))
+    )
+    (pad 1 smd rect (at -1.05 0) (size 0.6 0.45) (layers F.Cu F.Paste F.Mask)
+      (net 72 "Net-(BZ1-Pad1)"))
+    (pad 2 smd rect (at 1.05 0) (size 0.6 0.45) (layers F.Cu F.Paste F.Mask)
+      (net 70 "Net-(BZ1-Pad2)"))
+    (model ${KISYS3DMOD}/Diode_SMD.3dshapes/D_SOD-323.wrl
+      (at (xyz 0 0 0))
+      (scale (xyz 1 1 1))

Commit message: Arrange components
Parts:
- moved D5 60.8 mm to (110.7, 104.6), turned to 90 degrees
- moved BZ1 58.3 mm to (106.9, 105.0)
- moved Q1 31.3 mm to (113.8, 100.1), turned to 90 degrees
- moved J10 19.1 mm to (132.8, 110.2), turned to 0 degrees
- moved J9 11.5 mm to (128.0, 98.6)
- moved R2 2.16 mm to (116.4, 97.5)
Changed lines of the file:
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@@
   )
   (module Connector:Tag-Connect_TC2030-IDC-NL_2x03_P1.27mm_Vertical (layer B.Cu)
-    (at 115.765 118.7 270)
+    (at 132.842 110.236)
     (descr "Tag-Connect programming header; http://www.tag-connect.com/Materials/TC2030-IDC-NL.pdf")
     (tags "tag connect programming header pogo pins")
     (attr virtual)
-    (fp_text reference J10 (at 0 -2.7 270) (layer B.Fab) hide
+    (fp_text reference J10 (at 0 -2.7 180) (layer B.Fab) hide
       (effects (font (size 0.3 0.3) (thickness 0.04)) (justify mirror))
     )
-    (fp_text value TC2030_NL (at 0.141 -1.661 270) (layer Cmts.User)
+    (fp_text value TC2030_NL (at 0.141 -1.661 180) (layer Cmts.User)
       (effects (font (size 0.3 0.3) (thickness 0.04)))
     )
@@
     (fp_line (start -1.27 -1.27) (end -1.905 -1.27) (layer B.SilkS) (width 0.12))
     (fp_line (start -1.905 -1.27) (end -1.905 -0.635) (layer B.SilkS) (width 0.12))
-    (fp_text user KEEPOUT (at 0 0 270) (layer Cmts.User)
+    (fp_text user KEEPOUT (at 0 0 180) (layer Cmts.User)
       (effects (font (size 0.4 0.4) (thickness 0.07)))
     )
-    (fp_text user %R (at -0.254 0 270) (layer Cmts.User)
+    (fp_text user %R (at -0.254 0 180) (layer Cmts.User)
       (effects (font (size 0.3 0.3) (thickness 0.04)))
     )
-    (pad 6 connect circle (at 1.27 0.635 270) (size 0.7874 0.7874) (layers B.Cu B.Mask)
+    (pad 6 connect circle (at 1.27 0.635) (size 0.7874 0.7874) (layers B.Cu B.Mask)
       (net 49 +5VB))
-    (pad 5 connect circle (at 1.27 -0.635 270) (size 0.7874 0.7874) (layers B.Cu B.Mask)
+    (pad 5 connect circle (at 1.27 -0.635) (size 0.7874 0.7874) (layers B.Cu B.Mask)
       (net 19 /Bottom/MOSI))
-    (pad 4 connect circle (at 0 0.635 270) (size 0.7874 0.7874) (layers B.Cu B.Mask)
+    (pad 4 connect circle (at 0 0.635) (size 0.7874 0.7874) (layers B.Cu B.Mask)
       (net 20 /Bottom/MISO))
-    (pad 3 connect circle (at 0 -0.635 270) (size 0.7874 0.7874) (layers B.Cu B.Mask)
+    (pad 3 connect circle (at 0 -0.635) (size 0.7874 0.7874) (layers B.Cu B.Mask)
       (net 21 /Bottom/SCK))
-    (pad 2 connect circle (at -1.27 0.635 270) (size 0.7874 0.7874) (layers B.Cu B.Mask)
+    (pad 2 connect circle (at -1.27 0.635) (size 0.7874 0.7874) (layers B.Cu B.Mask)
       (net 22 /Bottom/~RST))
-    (pad 1 connect circle (at -1.27 -0.635 270) (size 0.7874 0.7874) (layers B.Cu B.Mask)
+    (pad 1 connect circle (at -1.27 -0.635) (size 0.7874 0.7874) (layers B.Cu B.Mask)
       (net 50 GNDB))
-    (pad "" np_thru_hole circle (at -2.54 0 270) (size 0.9906 0.9906) (drill 0.9906) (layers *.Cu *.Mask))
-    (pad "" np_thru_hole circle (at 2.54 -1.016 270) (size 0.9906 0.9906) (drill 0.9906) (layers *.Cu *.Mask))
-    (pad "" np_thru_hole circle (at 2.54 1.016 270) (size 0.9906 0.9906) (drill 0.9906) (layers *.Cu *.Mask))
+    (pad "" np_thru_hole circle (at -2.54 0) (size 0.9906 0.9906) (drill 0.9906) (layers *.Cu *.Mask))
+    (pad "" np_thru_hole circle (at 2.54 -1.016) (size 0.9906 0.9906) (drill 0.9906) (layers *.Cu *.Mask))
+    (pad "" np_thru_hole circle (at 2.54 1.016) (size 0.9906 0.9906) (drill 0.9906) (layers *.Cu *.Mask))
   )
   (module Resistor_SMD:R_0402_1005Metric (layer F.Cu)
@@
   )
   (module Resistor_SMD:R_0402_1005Metric (layer F.Cu)
-    (at 115.04 99.247)
+    (at 116.355 97.536)
     (descr "Resistor SMD 0402 (1005 Metric), square (rectangular) end terminal, IPC_7351 nominal, (Body size source: http://www.tortai-tech.com/upload/download/2011102023233369053.pdf), generated with kicad-footprint-generator")
     (tags resistor)
@@
   )
   (module Connector_PinHeader_2.54mm:PinHeader_1x01_P2.54mm_Vertical (layer F.Cu)
-    (at 127.082 110.042)
+    (at 128.016 98.552)
     (descr "Through hole straight pin header, 1x01, 2.54mm pitch, single row")
     (tags "Through hole pin header THT 1x01 2.54mm single row")
@@
   )
   (module Package_TO_SOT_SMD:SOT-23 (layer F.Cu)
-    (at 130.556 73.66)
+    (at 113.792 100.076 90)
     (descr "SOT-23, Standard")
     (tags SOT-23)
     (attr smd)
-    (fp_text reference Q1 (at 0 -2.5) (layer F.SilkS)
-      (effects (font (size 1 1) (thickness 0.15)))
-    )
-    (fp_text value 2N3904 (at 0 2.5) (layer F.Fab)
+    (fp_text reference Q1 (at 0 -2.5 90) (layer F.SilkS)
+      (effects (font (size 1 1) (thickness 0.15)))
+    )
+    (fp_text value 2N3904 (at 0 2.5 90) (layer F.Fab)
       (effects (font (size 1 1) (thickness 0.15)))
     )
@@
     (fp_line (start -0.15 -1.52) (end 0.7 -1.52) (layer F.Fab) (width 0.1))
     (fp_line (start -0.7 -0.95) (end -0.7 1.5) (layer F.Fab) (width 0.1))
-    (fp_text user %R (at 0 0 90) (layer F.Fab)
+    (fp_text user %R (at 0 0) (layer F.Fab)
       (effects (font (size 0.5 0.5) (thickness 0.075)))
     )
-    (pad 1 smd rect (at -1 -0.95) (size 0.9 0.8) (layers F.Cu F.Paste F.Mask)
+    (pad 1 smd rect (at -1 -0.95 90) (size 0.9 0.8) (layers F.Cu F.Paste F.Mask)
       (net 50 GNDB))
-    (pad 2 smd rect (at -1 0.95) (size 0.9 0.8) (layers F.Cu F.Paste F.Mask)
+    (pad 2 smd rect (at -1 0.95 90) (size 0.9 0.8) (layers F.Cu F.Paste F.Mask)
       (net 69 "Net-(Q1-Pad2)"))
-    (pad 3 smd rect (at 1 0) (size 0.9 0.8) (layers F.Cu F.Paste F.Mask)
+    (pad 3 smd rect (at 1 0 90) (size 0.9 0.8) (layers F.Cu F.Paste F.Mask)
       (net 70 "Net-(BZ1-Pad2)"))
     (model ${KISYS3DMOD}/Package_TO_SOT_SMD.3dshapes/SOT-23.wrl
@@
   )
   (module node:MLT-5020 (layer F.Cu)
-    (at 143.2 59.302001)
+    (at 106.934 105)
     (fp_text reference BZ1 (at 0 -3.4) (layer F.SilkS)
       (effects (font (size 1 1) (thickness 0.15)))
@@
   )
   (module Diode_SMD:D_SOD-323 (layer F.Cu)
-    (at 149.325001 57.617001)
+    (at 110.744 104.648 90)
     (descr SOD-323)
     (tags SOD-323)
     (attr smd)
-    (fp_text reference D5 (at 0 -1.85) (layer F.SilkS)
-      (effects (font (size 1 1) (thickness 0.15)))
-    )
-    (fp_text value 1N4148 (at 0.1 1.9) (layer F.Fab)
+    (fp_text reference D5 (at 0 -1.85 90) (layer F.SilkS)
+      (effects (font (size 1 1) (thickness 0.15)))
+    )
+    (fp_text value 1N4148 (at 0.1 1.9 90) (layer F.Fab)
       (effects (font (size 1 1) (thickness 0.15)))
     )
@@
     (fp_line (start 0.2 0) (end 0.45 0) (layer F.Fab) (width 0.1))
     (fp_line (start -1.5 -0.85) (end -1.5 0.85) (layer F.SilkS) (width 0.12))
-    (fp_text user %R (at 0 -1.85) (layer F.Fab)
-      (effects (font (size 1 1) (thickness 0.15)))
-    )
-    (pad 1 smd rect (at -1.05 0) (size 0.6 0.45) (layers F.Cu F.Paste F.Mask)
+    (fp_text user %R (at 0 -1.85 90) (layer F.Fab)
+      (effects (font (size 1 1) (thickness 0.15)))
+    )
+    (pad 1 smd rect (at -1.05 0 90) (size 0.6 0.45) (layers F.Cu F.Paste F.Mask)
       (net 72 "Net-(BZ1-Pad1)"))
-    (pad 2 smd rect (at 1.05 0) (size 0.6 0.45) (layers F.Cu F.Paste F.Mask)
+    (pad 2 smd rect (at 1.05 0 90) (size 0.6 0.45) (layers F.Cu F.Paste F.Mask)
       (net 70 "Net-(BZ1-Pad2)"))
     (model ${KISYS3DMOD}/Diode_SMD.3dshapes/D_SOD-323.wrl
