File: pcb/draft.kicad_pcb (KiCad board)
At the start: 2 copper layers, 109 x 54 mm, 62 parts, among them J1 MALE, J10 TC2030_NL, J101 MALE, J102 FEMALE, J103 MALE, J104 FEMALE, J105 MALE, J106 FEMALE, J107 MALE, J108 FEMALE, J11 STANDOFF, J111 STANDOFF, J112 STANDOFF, J113 STANDOFF, J114 STANDOFF, J12 STANDOFF, J13 STANDOFF, J14 STANDOFF, J2 FEMALE, J3 MALE, J4 FEMALE, J5 MALE, J6 FEMALE, J7 MALE, J8 FEMALE, J9 DTR, Q1 2N3904, SW1 ACTION, SW2 ACTION, SW3 ACTION, SW4 ACTION, U3 ATmega328P-MU, Y1 YSX321SL

Commit message: Play with shape / design
Parts:
- added REF**: Leaf, node:Leaf, F.Cu at (194.0, 123.0)
- moved R16 68.9 mm to (111.5, 110.0)
- moved R13 65.5 mm to (132.5, 115.0)
- moved R12 61.5 mm to (132.0, 92.5)
- moved R14 48.0 mm to (110.5, 117.5)
- moved R15 38.7 mm to (115.5, 102.5)
- moved J112 25.3 mm to (188.7, 92.3)
- moved J113 25.3 mm to (188.7, 117.7)
- moved R11 23.4 mm to (110.0, 95.0)
- moved R10 4.95 mm to (105.1, 95.5)
- moved BZ1 0.07 mm to (107.0, 105.0)
- turned SW1 to 135 degrees
- turned SW2 to 45 degrees
- turned SW3 to 315 degrees
- turned SW4 to 225 degrees
Routing:
- net Net-(J112-Pad1): track 0.00 -> 22.0 mm
- net Net-(J114-Pad1): track 0.00 -> 16.6 mm
- net Net-(J111-Pad1): track 0.00 -> 16.6 mm
- net GND: track 0.00 -> 15.9 mm, vias 0 -> 1
- net Net-(J113-Pad1): track 0.00 -> 4.38 mm
- added copper zone on B.Cu, net GND
- added copper zone on F.Cu, net GND
