File: pcb/top.sch (KiCad schematic (older format))
At the start: 16 parts, among them J101 MALE, J102 FEMALE, J103 MALE, J104 FEMALE, J105 MALE, J106 FEMALE, J107 MALE, J108 FEMALE, J111 STANDOFF, J112 STANDOFF, J113 STANDOFF, J114 STANDOFF, SW1 ACTION, SW2 ACTION, SW3 ACTION, SW4 ACTION

Commit message: Iterate
Parts:
- SW1, SW2, SW3, SW4: LCSC Part # C412374 -> C318884; MPN TS4560TP -> TS-1187A-B-A-B; Manufacturer SHOU HAN -> XKB Connectivity
Changed lines of the file:
@@
 $Descr A4 11693 8268
 encoding utf-8
-Sheet 2 3
+Sheet 3 3
 Title "Top"
 Date ""
@@
 F 1 "ACTION" H 2900 4394 50  0000 C CNN
 F 2 "Button_Switch_SMD:SW_SPST_TL3305A" H 2900 4400 50  0001 C CNN
-F 3 "https://datasheet.lcsc.com/szlcsc/1912111437_SHOU-HAN-TS4560TP_C412374.pdf" H 2900 4400 50  0001 C CNN
-F 4 "C412374" H 2900 4200 50  0001 C CNN "LCSC Part #"
-F 5 "TS4560TP" H 2900 4200 50  0001 C CNN "MPN"
-F 6 "SHOU HAN" H 2900 4200 50  0001 C CNN "Manufacturer"
+F 3 "https://datasheet.lcsc.com/szlcsc/2002271431_XKB-Connectivity-TS-1187A-B-A-B_C318884.pdf" H 2900 4400 50  0001 C CNN
+F 4 "C318884" H 2900 4200 50  0001 C CNN "LCSC Part #"
+F 5 "TS-1187A-B-A-B" H 2900 4200 50  0001 C CNN "MPN"
+F 6 "XKB Connectivity" H 2900 4200 50  0001 C CNN "Manufacturer"
 	1    2900 4200
 	1    0    0    -1
@@
 F 1 "ACTION" H 4400 4394 50  0000 C CNN
 F 2 "Button_Switch_SMD:SW_SPST_TL3305A" H 4400 4400 50  0001 C CNN
-F 3 "https://datasheet.lcsc.com/szlcsc/1912111437_SHOU-HAN-TS4560TP_C412374.pdf" H 4400 4400 50  0001 C CNN
-F 4 "C412374" H 4400 4200 50  0001 C CNN "LCSC Part #"
-F 5 "TS4560TP" H 4400 4200 50  0001 C CNN "MPN"
-F 6 "SHOU HAN" H 4400 4200 50  0001 C CNN "Manufacturer"
+F 3 "https://datasheet.lcsc.com/szlcsc/2002271431_XKB-Connectivity-TS-1187A-B-A-B_C318884.pdf" H 4400 4400 50  0001 C CNN
+F 4 "C318884" H 4400 4200 50  0001 C CNN "LCSC Part #"
+F 5 "TS-1187A-B-A-B" H 4400 4200 50  0001 C CNN "MPN"
+F 6 "XKB Connectivity" H 4400 4200 50  0001 C CNN "Manufacturer"
 	1    4400 4200
 	1    0    0    -1
@@
 F 1 "ACTION" H 5900 4394 50  0000 C CNN
 F 2 "Button_Switch_SMD:SW_SPST_TL3305A" H 5900 4400 50  0001 C CNN
-F 3 "https://datasheet.lcsc.com/szlcsc/1912111437_SHOU-HAN-TS4560TP_C412374.pdf" H 5900 4400 50  0001 C CNN
-F 4 "C412374" H 5900 4200 50  0001 C CNN "LCSC Part #"
-F 5 "TS4560TP" H 5900 4200 50  0001 C CNN "MPN"
-F 6 "SHOU HAN" H 5900 4200 50  0001 C CNN "Manufacturer"
+F 3 "https://datasheet.lcsc.com/szlcsc/2002271431_XKB-Connectivity-TS-1187A-B-A-B_C318884.pdf" H 5900 4400 50  0001 C CNN
+F 4 "C318884" H 5900 4200 50  0001 C CNN "LCSC Part #"
+F 5 "TS-1187A-B-A-B" H 5900 4200 50  0001 C CNN "MPN"
+F 6 "XKB Connectivity" H 5900 4200 50  0001 C CNN "Manufacturer"
 	1    5900 4200
 	1    0    0    -1
@@
 F 1 "ACTION" H 7400 4394 50  0000 C CNN
 F 2 "Button_Switch_SMD:SW_SPST_TL3305A" H 7400 4400 50  0001 C CNN
-F 3 "https://datasheet.lcsc.com/szlcsc/1912111437_SHOU-HAN-TS4560TP_C412374.pdf" H 7400 4400 50  0001 C CNN
-F 4 "C412374" H 7400 4200 50  0001 C CNN "LCSC Part #"
-F 5 "TS4560TP" H 7400 4200 50  0001 C CNN "MPN"
-F 6 "SHOU HAN" H 7400 4200 50  0001 C CNN "Manufacturer"
+F 3 "https://datasheet.lcsc.com/szlcsc/2002271431_XKB-Connectivity-TS-1187A-B-A-B_C318884.pdf" H 7400 4400 50  0001 C CNN
+F 4 "C318884" H 7400 4200 50  0001 C CNN "LCSC Part #"
+F 5 "TS-1187A-B-A-B" H 7400 4200 50  0001 C CNN "MPN"
+F 6 "XKB Connectivity" H 7400 4200 50  0001 C CNN "Manufacturer"
 	1    7400 4200
 	1    0    0    -1

Commit message: Update
Parts:
- SW1, SW2, SW3, SW4: footprint Button_Switch_SMD:SW_SPST_TL3305A -> node:TS-1187A-B-A-B
Changed lines of the file:
@@
 F 0 "SW1" H 2900 4485 50  0000 C CNN
 F 1 "ACTION" H 2900 4394 50  0000 C CNN
-F 2 "Button_Switch_SMD:SW_SPST_TL3305A" H 2900 4400 50  0001 C CNN
+F 2 "node:TS-1187A-B-A-B" H 2900 4400 50  0001 C CNN
 F 3 "https://datasheet.lcsc.com/szlcsc/2002271431_XKB-Connectivity-TS-1187A-B-A-B_C318884.pdf" H 2900 4400 50  0001 C CNN
 F 4 "C318884" H 2900 4200 50  0001 C CNN "LCSC Part #"
@@
 F 0 "SW2" H 4400 4485 50  0000 C CNN
 F 1 "ACTION" H 4400 4394 50  0000 C CNN
-F 2 "Button_Switch_SMD:SW_SPST_TL3305A" H 4400 4400 50  0001 C CNN
+F 2 "node:TS-1187A-B-A-B" H 4400 4400 50  0001 C CNN
 F 3 "https://datasheet.lcsc.com/szlcsc/2002271431_XKB-Connectivity-TS-1187A-B-A-B_C318884.pdf" H 4400 4400 50  0001 C CNN
 F 4 "C318884" H 4400 4200 50  0001 C CNN "LCSC Part #"
@@
 F 0 "SW3" H 5900 4485 50  0000 C CNN
 F 1 "ACTION" H 5900 4394 50  0000 C CNN
-F 2 "Button_Switch_SMD:SW_SPST_TL3305A" H 5900 4400 50  0001 C CNN
+F 2 "node:TS-1187A-B-A-B" H 5900 4400 50  0001 C CNN
 F 3 "https://datasheet.lcsc.com/szlcsc/2002271431_XKB-Connectivity-TS-1187A-B-A-B_C318884.pdf" H 5900 4400 50  0001 C CNN
 F 4 "C318884" H 5900 4200 50  0001 C CNN "LCSC Part #"
@@
 F 0 "SW4" H 7400 4485 50  0000 C CNN
 F 1 "ACTION" H 7400 4394 50  0000 C CNN
-F 2 "Button_Switch_SMD:SW_SPST_TL3305A" H 7400 4400 50  0001 C CNN
+F 2 "node:TS-1187A-B-A-B" H 7400 4400 50  0001 C CNN
 F 3 "https://datasheet.lcsc.com/szlcsc/2002271431_XKB-Connectivity-TS-1187A-B-A-B_C318884.pdf" H 7400 4400 50  0001 C CNN
 F 4 "C318884" H 7400 4200 50  0001 C CNN "LCSC Part #"

Commit message: Update solder mask keep out
Parts:
- SW1, SW2, SW3, SW4: footprint node:TS-1187A-B-A-B -> node:top-leaf
Changed lines of the file:
@@
 F 0 "SW1" H 2900 4485 50  0000 C CNN
 F 1 "ACTION" H 2900 4394 50  0000 C CNN
-F 2 "node:TS-1187A-B-A-B" H 2900 4400 50  0001 C CNN
+F 2 "node:top-leaf" H 2900 4400 50  0001 C CNN
 F 3 "https://datasheet.lcsc.com/szlcsc/2002271431_XKB-Connectivity-TS-1187A-B-A-B_C318884.pdf" H 2900 4400 50  0001 C CNN
 F 4 "C318884" H 2900 4200 50  0001 C CNN "LCSC Part #"
@@
 F 0 "SW2" H 4400 4485 50  0000 C CNN
 F 1 "ACTION" H 4400 4394 50  0000 C CNN
-F 2 "node:TS-1187A-B-A-B" H 4400 4400 50  0001 C CNN
+F 2 "node:top-leaf" H 4400 4400 50  0001 C CNN
 F 3 "https://datasheet.lcsc.com/szlcsc/2002271431_XKB-Connectivity-TS-1187A-B-A-B_C318884.pdf" H 4400 4400 50  0001 C CNN
 F 4 "C318884" H 4400 4200 50  0001 C CNN "LCSC Part #"
@@
 F 0 "SW3" H 5900 4485 50  0000 C CNN
 F 1 "ACTION" H 5900 4394 50  0000 C CNN
-F 2 "node:TS-1187A-B-A-B" H 5900 4400 50  0001 C CNN
+F 2 "node:top-leaf" H 5900 4400 50  0001 C CNN
 F 3 "https://datasheet.lcsc.com/szlcsc/2002271431_XKB-Connectivity-TS-1187A-B-A-B_C318884.pdf" H 5900 4400 50  0001 C CNN
 F 4 "C318884" H 5900 4200 50  0001 C CNN "LCSC Part #"
@@
 F 0 "SW4" H 7400 4485 50  0000 C CNN
 F 1 "ACTION" H 7400 4394 50  0000 C CNN
-F 2 "node:TS-1187A-B-A-B" H 7400 4400 50  0001 C CNN
+F 2 "node:top-leaf" H 7400 4400 50  0001 C CNN
 F 3 "https://datasheet.lcsc.com/szlcsc/2002271431_XKB-Connectivity-TS-1187A-B-A-B_C318884.pdf" H 7400 4400 50  0001 C CNN
 F 4 "C318884" H 7400 4200 50  0001 C CNN "LCSC Part #"

Commit message: Add +5V network
Connections:
- net +5V: now reaches J101.1 (Pin_1), J102.1 (Pin_1)
- net +5V: now also J103.1 (Pin_1), J104.1 (Pin_1), J105.1 (Pin_1), J106.1 (Pin_1), J107.1 (Pin_1), J108.1 (Pin_1)
Changed lines of the file:
@@
 Wire Wire Line
 	2500 2550 2500 2750
+$Comp
+L power:+5V #PWR?
+U 1 1 5F924455
+P 4300 2050
+F 0 "#PWR?" H 4300 1900 50  0001 C CNN
+F 1 "+5V" H 4315 2223 50  0000 C CNN
+F 2 "" H 4300 2050 50  0001 C CNN
+F 3 "" H 4300 2050 50  0001 C CNN
+	1    4300 2050
+	1    0    0    -1
+$EndComp
+$Comp
+L power:+5V #PWR?
+U 1 1 5F924519
+P 5100 2050
+F 0 "#PWR?" H 5100 1900 50  0001 C CNN
+F 1 "+5V" H 5115 2223 50  0000 C CNN
+F 2 "" H 5100 2050 50  0001 C CNN
+F 3 "" H 5100 2050 50  0001 C CNN
+	1    5100 2050
+	1    0    0    -1
+$EndComp
+$Comp
+L power:+5V #PWR?
+U 1 1 5F92463C
+P 5900 2050
+F 0 "#PWR?" H 5900 1900 50  0001 C CNN
+F 1 "+5V" H 5915 2223 50  0000 C CNN
+F 2 "" H 5900 2050 50  0001 C CNN
+F 3 "" H 5900 2050 50  0001 C CNN
+	1    5900 2050
+	1    0    0    -1
+$EndComp
+$Comp
+L power:+5V #PWR?
+U 1 1 5F9242A3
+P 3500 2050
+F 0 "#PWR?" H 3500 1900 50  0001 C CNN
+F 1 "+5V" H 3515 2223 50  0000 C CNN
+F 2 "" H 3500 2050 50  0001 C CNN
+F 3 "" H 3500 2050 50  0001 C CNN
+	1    3500 2050
+	1    0    0    -1
+$EndComp
+Wire Wire Line
+	3500 2050 3500 2100
+Connection ~ 3500 2100
+Wire Wire Line
+	4300 2050 4300 2100
+Connection ~ 4300 2100
+Wire Wire Line
+	5100 2050 5100 2100
+Connection ~ 5100 2100
+Wire Wire Line
+	5900 2100 5900 2050
+Connection ~ 5900 2100
+$Comp
+L power:+5V #PWR?
+U 1 1 5F92BE15
+P 2900 2550
+F 0 "#PWR?" H 2900 2400 50  0001 C CNN
+F 1 "+5V" H 2915 2723 50  0000 C CNN
+F 2 "" H 2900 2550 50  0001 C CNN
+F 3 "" H 2900 2550 50  0001 C CNN
+	1    2900 2550
+	1    0    0    -1
+$EndComp
+$Comp
+L power:PWR_FLAG #FLG?
+U 1 1 5F92BF03
+P 2900 2750
+F 0 "#FLG?" H 2900 2825 50  0001 C CNN
+F 1 "PWR_FLAG" H 2900 2923 50  0000 C CNN
+F 2 "" H 2900 2750 50  0001 C CNN
+F 3 "~" H 2900 2750 50  0001 C CNN
+	1    2900 2750
+	-1   0    0    1
+$EndComp
+Wire Wire Line
+	2900 2750 2900 2550
 $EndSCHEMATC
