File: pcb/bottom.sch (KiCad schematic (older format))
At the start: 42 parts, among them J1 MALE, J10 TC2030_NL, J11 STANDOFF, J12 STANDOFF, J13 STANDOFF, J14 STANDOFF, J2 FEMALE, J3 MALE, J4 FEMALE, J5 MALE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

Commit message: Switch to WS2813C (bigger footprint)
Parts:
- D1, D2, D3, D4: LCSC Part # C189639 -> C194323; MPN WS2813-Mini(WS2813-3535) -> WS2813C
Changed lines of the file:
@@
 F 1 "WS2813" H 4800 3400 50  0000 L CNN
 F 2 "node:WS2813-Mini" H 4800 2850 50  0001 L TNN
-F 3 "https://datasheet.lcsc.com/szlcsc/1810010024_Worldsemi-WS2813-Mini-WS2813-3535_C189639.pdf" H 4850 2775 50  0001 L TNN
-F 4 "C189639" H 4750 3150 50  0001 C CNN "LCSC Part #"
-F 5 "WS2813-Mini(WS2813-3535)" H 4750 3150 50  0001 C CNN "MPN"
+F 3 "https://datasheet.lcsc.com/szlcsc/1809291530_Worldsemi-WS2813C_C194323.pdf" H 4850 2775 50  0001 L TNN
+F 4 "C194323" H 4750 3150 50  0001 C CNN "LCSC Part #"
+F 5 "WS2813C" H 4750 3150 50  0001 C CNN "MPN"
 F 6 "Worldsemi" H 4750 3150 50  0001 C CNN "Manufacturer"
 	1    4750 3150
@@
 F 1 "WS2813" H 5600 3400 50  0000 L CNN
 F 2 "node:WS2813-Mini" H 5600 2850 50  0001 L TNN
-F 3 "https://datasheet.lcsc.com/szlcsc/1810010024_Worldsemi-WS2813-Mini-WS2813-3535_C189639.pdf" H 5650 2775 50  0001 L TNN
-F 4 "C189639" H 5550 3150 50  0001 C CNN "LCSC Part #"
-F 5 "WS2813-Mini(WS2813-3535)" H 5550 3150 50  0001 C CNN "MPN"
+F 3 "https://datasheet.lcsc.com/szlcsc/1809291530_Worldsemi-WS2813C_C194323.pdf" H 5650 2775 50  0001 L TNN
+F 4 "C194323" H 5550 3150 50  0001 C CNN "LCSC Part #"
+F 5 "WS2813C" H 5550 3150 50  0001 C CNN "MPN"
 F 6 "Worldsemi" H 5550 3150 50  0001 C CNN "Manufacturer"
 	1    5550 3150
@@
 F 1 "WS2813" H 6400 3400 50  0000 L CNN
 F 2 "node:WS2813-Mini" H 6400 2850 50  0001 L TNN
-F 3 "https://datasheet.lcsc.com/szlcsc/1810010024_Worldsemi-WS2813-Mini-WS2813-3535_C189639.pdf" H 6450 2775 50  0001 L TNN
-F 4 "C189639" H 6350 3150 50  0001 C CNN "LCSC Part #"
-F 5 "WS2813-Mini(WS2813-3535)" H 6350 3150 50  0001 C CNN "MPN"
+F 3 "https://datasheet.lcsc.com/szlcsc/1809291530_Worldsemi-WS2813C_C194323.pdf" H 6450 2775 50  0001 L TNN
+F 4 "C194323" H 6350 3150 50  0001 C CNN "LCSC Part #"
+F 5 "WS2813C" H 6350 3150 50  0001 C CNN "MPN"
 F 6 "Worldsemi" H 6350 3150 50  0001 C CNN "Manufacturer"
 	1    6350 3150
@@
 F 1 "WS2813" H 7200 3400 50  0000 L CNN
 F 2 "node:WS2813-Mini" H 7200 2850 50  0001 L TNN
-F 3 "https://datasheet.lcsc.com/szlcsc/1810010024_Worldsemi-WS2813-Mini-WS2813-3535_C189639.pdf" H 7250 2775 50  0001 L TNN
-F 4 "C189639" H 7150 3150 50  0001 C CNN "LCSC Part #"
-F 5 "WS2813-Mini(WS2813-3535)" H 7150 3150 50  0001 C CNN "MPN"
+F 3 "https://datasheet.lcsc.com/szlcsc/1809291530_Worldsemi-WS2813C_C194323.pdf" H 7250 2775 50  0001 L TNN
+F 4 "C194323" H 7150 3150 50  0001 C CNN "LCSC Part #"
+F 5 "WS2813C" H 7150 3150 50  0001 C CNN "MPN"
 F 6 "Worldsemi" H 7150 3150 50  0001 C CNN "Manufacturer"
 	1    7150 3150

Commit message: Assign bottom-leaf footprints to LEDs
Parts:
- D1, D2, D3, D4: footprint node:WS2813-Mini -> node:bottom-leaf
Other:
- note added: "https://electronics.stackexchange.com/q/527338/21817"
- note removed: "Maybe rework, see:\nhttps://electronics.stackexchange.com/q/527338/21817"
Changed lines of the file:
@@
 F 0 "D1" H 4800 3500 50  0000 L CNN
 F 1 "WS2813" H 4800 3400 50  0000 L CNN
-F 2 "node:WS2813-Mini" H 4800 2850 50  0001 L TNN
+F 2 "node:bottom-leaf" H 4800 2850 50  0001 L TNN
 F 3 "https://datasheet.lcsc.com/szlcsc/1809291530_Worldsemi-WS2813C_C194323.pdf" H 4850 2775 50  0001 L TNN
 F 4 "C194323" H 4750 3150 50  0001 C CNN "LCSC Part #"
@@
 F 0 "D2" H 5600 3500 50  0000 L CNN
 F 1 "WS2813" H 5600 3400 50  0000 L CNN
-F 2 "node:WS2813-Mini" H 5600 2850 50  0001 L TNN
+F 2 "node:bottom-leaf" H 5600 2850 50  0001 L TNN
 F 3 "https://datasheet.lcsc.com/szlcsc/1809291530_Worldsemi-WS2813C_C194323.pdf" H 5650 2775 50  0001 L TNN
 F 4 "C194323" H 5550 3150 50  0001 C CNN "LCSC Part #"
@@
 F 0 "D3" H 6400 3500 50  0000 L CNN
 F 1 "WS2813" H 6400 3400 50  0000 L CNN
-F 2 "node:WS2813-Mini" H 6400 2850 50  0001 L TNN
+F 2 "node:bottom-leaf" H 6400 2850 50  0001 L TNN
 F 3 "https://datasheet.lcsc.com/szlcsc/1809291530_Worldsemi-WS2813C_C194323.pdf" H 6450 2775 50  0001 L TNN
 F 4 "C194323" H 6350 3150 50  0001 C CNN "LCSC Part #"
@@
 F 0 "D4" H 7200 3500 50  0000 L CNN
 F 1 "WS2813" H 7200 3400 50  0000 L CNN
-F 2 "node:WS2813-Mini" H 7200 2850 50  0001 L TNN
+F 2 "node:bottom-leaf" H 7200 2850 50  0001 L TNN
 F 3 "https://datasheet.lcsc.com/szlcsc/1809291530_Worldsemi-WS2813C_C194323.pdf" H 7250 2775 50  0001 L TNN
 F 4 "C194323" H 7150 3150 50  0001 C CNN "LCSC Part #"
@@
 Wire Notes Line
 	7050 6100 7050 4100
-Text Notes 7050 6300 0    50   ~ 0
-Maybe rework, see:\nhttps://electronics.stackexchange.com/q/527338/21817
+Text Notes 7050 6200 0    50   ~ 0
+https://electronics.stackexchange.com/q/527338/21817
 $Comp
 L node:+5VB #PWR0107
