File: atom/lower.sch (KiCad schematic (older format))
At the start: 39 parts, among them J10 TC2030_NL, J11 STANDOFF, J12 STANDOFF, J13 STANDOFF, J14 STANDOFF, J2 FEMALE, J4 FEMALE, J6 FEMALE, J8 FEMALE, J9 DTR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

Commit message: Clean up and rename: PCB -> atom
Parts:
- U3: symbol draft-rescue:ATmega328P-MU-MCU_Microchip_ATmega -> MCU_Microchip_ATmega:ATmega328P-MU
Changed lines of the file:
@@
 $EndComp
 $Comp
-L draft-rescue:ATmega328P-MU-MCU_Microchip_ATmega U?
+L MCU_Microchip_ATmega:ATmega328P-MU U?
 U 1 1 5CAD6264
 P 1500 5900
