File: adapter/lower.sch (KiCad schematic (older format))
At the start: 14 parts, among them J2 FEMALE, J3 STANDOFF, J4 STANDOFF, J5 STANDOFF, J6 USB_C_Receptacle_USB2.0, J7 DTR, U1 FT232RL

Commit message: Swap RX/TX on lower board
Connections:
- net RXD: now also J2.2 (Pin_2); no longer J2.1 (Pin_1)
- net TXD: now also J2.1 (Pin_1); no longer J2.2 (Pin_2)
Changed lines of the file:
@@
 $EndComp
 Text Label 3050 1650 2    50   ~ 0
+TXD
+Text Label 3050 1750 2    50   ~ 0
 RXD
-Text Label 3050 1750 2    50   ~ 0
-TXD
 Wire Wire Line
 	3150 1650 3050 1650
@@
 	3650 1650 3750 1650
 $Comp
-L node:+5VB #PWR?
+L node:+5VB #PWR0105
 U 1 1 5FD11CF7
 P 3750 1600
-F 0 "#PWR?" H 3750 1450 50  0001 C CNN
+F 0 "#PWR0105" H 3750 1450 50  0001 C CNN
 F 1 "+5VB" H 3765 1773 50  0000 C CNN
 F 2 "" H 3750 1600 50  0001 C CNN
@@
 $EndComp
 $Comp
-L node:GNDB #PWR?
+L node:GNDB #PWR0106
 U 1 1 5FD11BCA
 P 3750 1800
-F 0 "#PWR?" H 3750 1550 50  0001 C CNN
+F 0 "#PWR0106" H 3750 1550 50  0001 C CNN
 F 1 "GNDB" H 3755 1627 50  0000 C CNN
 F 2 "" H 3750 1800 50  0001 C CNN
@@
 $EndComp
 $Comp
-L node:GNDB #PWR?
+L node:GNDB #PWR0107
 U 1 1 5FD33CC5
 P 3500 4250
-F 0 "#PWR?" H 3500 4000 50  0001 C CNN
+F 0 "#PWR0107" H 3500 4000 50  0001 C CNN
 F 1 "GNDB" H 3505 4077 50  0000 C CNN
 F 2 "" H 3500 4250 50  0001 C CNN
